File: output/pcbs/top_plate.kicad_pcb (KiCad board)
At the start: 2 copper layers, 122.3 x 101.1 mm, 39 parts

Commit message: Wip Makefile
Parts:
- removed MCU1, MCU2: , ProMicro
- removed REF**: TRRS-PJ-320A-dual, TRRS-PJ-320A-dual
Other:
- outline, holes or cut-outs redrawn
