File: output/pcbs/top_plate.kicad_pcb (KiCad board)
At the start: 2 copper layers, 122.3 x 101.1 mm, 36 parts

Commit message: A probably working version
Parts:
- removed D1, D10, D11, D12, D13, D14, D15, D16, D17, D18, D2, D3, D4, D5, D6, D7, D8, D9: , ComboDiode
- removed S1, S10, S11, S12, S13, S14, S15, S16, S17, S18, S2, S3, S4, S5, S6, S7, S8, S9: , PG1350
