File: output/pcbs/bottom_plate.kicad_pcb (KiCad board)
At the start: 2 copper layers, 122.3 x 101.1 mm, 36 parts

Commit message: wip
Other:
- net class Power added: clearance 0.2, trace_width 0.5, via_dia 0.8, via_drill 0.4
Changed lines of the file:
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@@
 (net 26 "home_thumb")
 (net 27 "far_thumb")
-  (net_class Default "This is the default net class."
+  (net_class Default "This is the default net class"
     (clearance 0.2)
     (trace_width 0.25)
@@
 (add_net "far_thumb")
   )
+  (net_class Power "This is the power net class"
+    (clearance 0.2)
+    (trace_width 0.5)
+    (via_dia 0.8)
+    (via_drill 0.4)
+    (uvia_dia 0.3)
+    (uvia_drill 0.1)
+  )
       (module PG1350 (layer F.Cu)

Commit message: A probably working version
Parts:
- removed D1, D10, D11, D12, D13, D14, D15, D16, D17, D18, D2, D3, D4, D5, D6, D7, D8, D9: , ComboDiode
- removed S1, S10, S11, S12, S13, S14, S15, S16, S17, S18, S2, S3, S4, S5, S6, S7, S8, S9: , PG1350
