File: output/pcbs/board.kicad_pcb (KiCad board)
At the start: 2 copper layers, 122.3 x 101.1 mm, 40 parts

Commit message: Minor progress
Parts:
- removed REF** (x2): TRRS-PJ-320A-dual, TRRS-PJ-320A-dual
- added TRRS1: TRRS-PJ-320A-dual, TRRS-PJ-320A-dual, F.Cu at (122.0, -0.20)
- added TRRS2: TRRS-PJ-320A-dual, TRRS-PJ-320A-dual, F.Cu at (122.0, -2.20)
Other:
- board text added: "samoklava v0.1 by soundmonster"
Changed lines of the file:
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@@
       (module TRRS-PJ-320A-dual (layer F.Cu)
       (at 122 -0.1999999999999993 270)
-      (fp_text reference REF** (at 0 14.2) (layer Dwgs.User) (effects (font (size 1 1) (thickness 0.15))))
+      (fp_text reference "TRRS1" (at 0 14.2) (layer Dwgs.User) (effects (font (size 1 1) (thickness 0.15))))
       (fp_text value TRRS-PJ-320A-dual (at 0 -5.6) (layer F.Fab) (effects (font (size 1 1) (thickness 0.15))))
       (fp_line (start 0.5 -2) (end -5.1 -2) (layer Dwgs.User) (width 0.15))
@@
       (module TRRS-PJ-320A-dual (layer F.Cu)
       (at 122 -2.1999999999999993 270)
-      (fp_text reference REF** (at 0 14.2) (layer Dwgs.User) (effects (font (size 1 1) (thickness 0.15))))
+      (fp_text reference "TRRS2" (at 0 14.2) (layer Dwgs.User) (effects (font (size 1 1) (thickness 0.15))))
       (fp_text value TRRS-PJ-320A-dual (at 0 -5.6) (layer F.Fab) (effects (font (size 1 1) (thickness 0.15))))
       (fp_line (start 0.5 -2) (end -5.1 -2) (layer Dwgs.User) (width 0.15))
@@
         (pad 4 thru_hole oval (at -4.6 3.2 270) (size 1.6 2.2) (drill oval 0.9 1.5) (layers *.Cu *.Mask) (net 36 "P0"))
       )
+            (gr_text "samoklava v0.1\nby soundmonster" (at 31.5 0 0) (layer F.SilkS)
+                (effects (font (size 1 1) (thickness 0.15)) (justify left))
+            )
+            (gr_text "samoklava v0.1\nby soundmonster" (at 31.5 0 0) (layer B.SilkS)
+                (effects (font (size 1 1) (thickness 0.15)) (justify right mirror))
+            )
             (gr_line (start 10 9.5) (end 26 9.5) (angle 90) (layer Edge.Cuts) (width 0.15))
 (gr_line (start 8 7.5) (end 8 -41.5) (angle 90) (layer Edge.Cuts) (width 0.15))

Commit message: wip
Parts:
- added B1, B2: , E73:SW_TACT_ALPS_SKQGABE010, F.Cu at (107.0, -10.2)
- added J1, J2: Jumper, lib:Jumper, F.Cu at (113.5, -10.2)
- added PAD1: , SMDPad, F.Cu at (113.0, -26.2)
- added PAD2: , SMDPad, F.Cu at (113.0, -29.2)
- added T1, T2: , E73:SPDT_C128955, F.Cu at (120.0, -10.2)
- moved TRRS1 5.00 mm to (122.0, 4.80)
- moved TRRS2 5.00 mm to (122.0, 2.80)
