File: output/routed_pcbs/bottom_plate.kicad_pcb (KiCad board)
At the start: 2 copper layers, 122.3 x 101.1 mm, 36 parts

Commit message: A probably working version
Parts:
- removed D1, D10, D11, D12, D13, D14, D15, D16, D17, D18, D2, D3, D4, D5, D6, D7, D8, D9: , ComboDiode
- removed S1, S10, S11, S12, S13, S14, S15, S16, S17, S18, S2, S3, S4, S5, S6, S7, S8, S9: , PG1350
Routing:
- net P19: track 173.1 -> 0.00 mm, vias 3 -> 0
- net P15: track 157.9 -> 0.00 mm, vias 2 -> 0
- net P18: track 150.5 -> 0.00 mm, vias 2 -> 0
- net P6: track 101.7 -> 0.00 mm
- net P7: track 97.8 -> 0.00 mm
- net P5: track 97.5 -> 0.00 mm
- net P20: track 86.0 -> 0.00 mm, vias 1 -> 0
- net P21: track 84.9 -> 0.00 mm, vias 2 -> 0
- net P4: track 49.3 -> 0.00 mm
- net near_thumb: track 41.1 -> 0.00 mm
- net home_thumb: track 30.3 -> 0.00 mm
- net far_thumb: track 29.6 -> 0.00 mm
- net pinky_bottom: track 29.4 -> 0.00 mm
- net index_top: track 29.1 -> 0.00 mm
- net index_home: track 29.1 -> 0.00 mm
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Other:
- net class Power added: clearance 0.2, trace_width 0.5, via_dia 0.8, via_drill 0.4
