File: output/routed_pcbs/top_plate.kicad_pcb (KiCad board)
At the start: 2 copper layers, 122.3 x 101.1 mm, 36 parts

Commit message: A probably working version
Parts:
- removed D1, D10, D11, D12, D13, D14, D15, D16, D17, D18, D2, D3, D4, D5, D6, D7, D8, D9: , ComboDiode
- removed S1, S10, S11, S12, S13, S14, S15, S16, S17, S18, S2, S3, S4, S5, S6, S7, S8, S9: , PG1350
Routing:
- net P15: track 171.4 -> 0.00 mm, vias 2 -> 0
- net P19: track 158.9 -> 0.00 mm, vias 2 -> 0
- net P18: track 148.5 -> 0.00 mm, vias 2 -> 0
- net P20: track 87.2 -> 0.00 mm, vias 1 -> 0
- net P21: track 84.4 -> 0.00 mm, vias 1 -> 0
Other:
- net class Power added: clearance 0.2, trace_width 0.5, via_dia 0.8, via_drill 0.4
